File: xiao led module.kicad_sch (KiCad schematic)
At the start: 52 parts, among them J2 Conn_01x04, U1 XIAO-ESP32-C3-DIP

Commit message: Source all BOM parts against live JLCPCB stock, generate fab files & docs
Re-sourced every part on the XIAO LED module board against the live
JLCPCB Open Platform API and generated complete, verified fabrication
files. The prior BOM/CPL (from Fabrication Toolkit) had an empty LCSC
Part # column, same issue seen on the esp32-c3-led board.

Part substitutions:
- D1-D50 (WS2812B-2020 LEDs): original part LCSC C965555 has only 4
  units in stock -- unusable for a 50-LED board. Replaced with
  XL-2020RGBC-2812B (C5349955, 127,770 in stock), confirmed via
  XINGLIGHT datasheet: same 2.0x2.0mm package, same VDD/GND/DI/DO
  pinout, WS2812-protocol compatible. Direct drop-in on the existing
  WS2812_2020 footprint.
- J2 (JST 4-pin connector): original part LCSC C265331 shows 0 units
  in stock. Replaced with WAFER-PH2.0-4PWB (C3029442, 45,426 in
  stock) -- same 4-pin, 2.0mm-pitch, right-angle SMD JST-PH-compatible
  connector, confirmed on the existing JST_1x04_P2.0mm_Horizontal_SMD
  footprint (pad pitch/geometry match).
- U1 (XIAO-ESP32-C3-DIP footprint): this is a SOCKET pattern (14 pads,
  2 rows x 7, 2.54mm pitch, both TH+SMD land per pad) for a pluggable
  XIAO module, not a direct-solder module footprint. JLCPCB has no
  machine-placeable 2.54mm female pin socket in their assembly
  catalog (known THT-socket limitation). Marked DNP
  (through_hole exclude_from_pos_files dnp) so it's correctly excluded
  from the BOM/CPL; board still gets the through-holes drilled for
  hand-soldering standard female headers post-fabrication.

Generated production/ fabrication set:
- bom.csv: JLCPCB-format BOM, 51 machine-assembled parts (50 LEDs +
  J2), U1 intentionally excluded per above
- positions.csv: CPL via ,
  verified 1:1 reference match against bom.csv
- gerbers/ + xiao_led_module_gerbers.zip: fresh Gerbers + Excellon
  drill export, ready to upload as-is
- Removed stale Fabrication Toolkit artifacts (netlist.ipc,
  designators.csv, old zip) that duplicated/conflicted with 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
Parts:
- D1, D10, D11, D12, D13, D14, D15, D16, D17, D18, D19, D2, D20, D21, D22, D23, D24, D25, D26, D27, D28, D29, D3, D30, D31, D32, D33, D34, D35, D36, D37, D38, D39, D4, D40, D41, D42, D43, D44, D45, D46, D47, D48, D49, D5, D50, D6, D7, D8, D9: LCSC (none) -> C5349955; MPN (none) -> XL-2020RGBC-2812B
- J2: LCSC (none) -> C3029442; MPN (none) -> WAFER-PH2.0-4PWB
- U1: MPN (none) -> DNP - hand-solder 2x 1x7 2.54mm female headers post-assembly
